File: DMH_Dual_VCF_Diode_Ladder_Mk2_PCB_1/Resonance_A_CV.kicad_sch (KiCad schematic)
At the start: 24 parts, among them Q1 BC548, Q2 BC548, U1 TL074

Commit message: Added board-to-board pins to schematic
Parts:
- added J17: Conn_01x10_PinHeader, Connector_PinHeader_2.54mm:PinHeader_1x10_P2.54mm_Vertical, symbol SynthStuff:Conn_01x10_PinHeader
Connections:
- net GND: now also J17.10 (Pin_10)
- net Res CV Input: now also J17.7 (Pin_7)
- net at R65.1, RV18.2: now also J17.9 (Pin_9)
- net at RV16.2, U1.12 (+): now also J17.8 (Pin_8)
