File: DMH_Dual_VCF_Diode_Ladder_Mk2_PCB_1/Core_Circuit_B.kicad_sch (KiCad schematic)
At the start: 41 parts, among them SW4 SW_SPDT, SW5 SW_SPDT, SW6 SW_SPDT, U4 TL074, U6 TL074

Commit message: Added board-to-board pins to schematic
Parts:
- added J18: Conn_01x10_PinHeader, Connector_PinHeader_2.54mm:PinHeader_1x10_P2.54mm_Vertical, symbol SynthStuff:Conn_01x10_PinHeader
Connections:
- net Input: now also J18.1 (Pin_1)
- net at C30.1, SW6.2 (B): now also J18.6 (Pin_6)
- net at C29.1, C31.1, SW5.2 (B): now also J18.5 (Pin_5)
- net at C28.1, RV14.2: now also J18.2 (Pin_2)
- net at SW4.1 (A), SW5.1 (A), SW6.1 (A)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: now also J18.3 (Pin_3)
- net at R49.1, R51.1, SW4.2 (B): now also J18.4 (Pin_4)

Commit message: Added inter-board pins to all circuits
Parts:
- removed unit 1 of J18
- removed unit 2 of J18
- removed RV14: 100k, SynthStuff:Potentiometer_Alpha_RD901F-40-00D_Single_Vertical, symbol Device:R_Potentiometer_US
- J20: renamed from J18; value Conn_01x10_PinHeader -> Conn_01x04_PinHeader; symbol SynthStuff:Conn_01x10_PinHeader -> SynthStuff:Conn_01x04_PinHeader
Connections:
- net Input: now also C28.1
- net at C30.1, SW6.2 (B): now also J20.4 (Pin_4); no longer J20.6 (Pin_6)
- net at SW4.1 (A), SW5.1 (A), SW6.1 (A)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: now also J20.1 (Pin_1); no longer J20.3 (Pin_3)
- net at C29.1, C31.1, SW5.2 (B): now also J20.3 (Pin_3); no longer J20.5 (Pin_5)
- net at R49.1, R51.1, SW4.2 (B): now also J20.2 (Pin_2); no longer J20.4 (Pin_4)
