File: DMH_Dual_VCF_Diode_Ladder_Mk2_PCB_1/Drive_B.kicad_sch (KiCad schematic)
At the start: 25 parts, among them J18 Conn_01x06_PinHeader, Q7 BC548, Q8 BC548, SW8 SW_DPDT_x2, U10 TL074

Commit message: Re-exported Gerbers
Parts:
- SW8: Function (none) -> Link D&R
Changed lines of the file:
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@@
 		(on_board no)
 		(dnp no)
-		(fields_autoplaced yes)
 		(property "Reference" "SW8"
 			(at 182.88 118.1099 90)
@@
 			)
 		)
+		(property "Function" "Link D&R"
+			(at 187.452 115.824 90)
+			(effects
+				(font
+					(size 1.27 1.27)
+					(thickness 0.254)
+					(bold yes)
+					(italic yes)
+				)
+			)
+		)
