File: DMH_Dual_VCF_Diode_Ladder_Mk2_PCB_2/DMH_Dual_VCF_Diode_Ladder_Mk2_PCB_2.kicad_pcb (KiCad board)
At the start: 2 copper layers, 146 x 175 mm, 70 parts, among them J15 Conn_01x08_PinHeader, J16 Conn_01x08_PinHeader, J17 Conn_01x06_PinHeader, J18 Conn_01x06_PinHeader, J19 Conn_01x06_PinHeader, J20 Conn_01x06_PinHeader, J21 Conn_01x06_PinHeader, J22 Conn_01x06_PinHeader, J23 Conn_01x04_PinHeader, SW1 SW_SPDT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

Commit message: Finished Mk2.0
Connections:
- R10 pad 1: Net-(SW7-A) -> Net-(SW7-C)
- R10 pad 2: Net-(SW7-C) -> Net-(SW7-A)
- R24 pad 1: Net-(SW9-A) -> Net-(SW9-C)
- R24 pad 2: Net-(SW9-C) -> Net-(SW9-A)
- RV19 pad 2: Net-(SW7-C) -> Net-(SW7-A)
- RV31 pad 2: Net-(SW9-C) -> Net-(SW9-A)
Routing:
- net Net-(SW7-A): track 108.9 -> 100.5 mm
- net Net-(J18B-Pin_2): track 168.9 -> 161.9 mm
- net Net-(J18C-Pin_3): track 162.6 -> 155.7 mm
- net /Drive A/Drive CV: track 156.3 -> 149.4 mm
- net Net-(SW7-C): track 82.1 -> 85.3 mm
- net Net-(SW9-B): track 105.6 -> 102.8 mm
- net Net-(SW9-C): track 94.4 -> 93.0 mm
- net Net-(SW9-A): track 105.5 -> 106.1 mm
Other:
- board text added: "Mk2.0 - March 2025"
- board text removed: "Mk2.0 - Month Year"
