File: DMH_Dual_VCF_Diode_Ladder_Mk2_PCB_2/Drive_A.kicad_sch (KiCad schematic)
At the start: 25 parts, among them J17 Conn_01x06_PinHeader, Q5 BC548, Q6 BC548, U9 TL074

Commit message: Complete Exclude From Board on PCB 2
Parts:
- J17: footprint Connector_PinHeader_2.54mm:PinHeader_1x06_P2.54mm_Vertical -> Connector_PinSocket_2.54mm:PinSocket_1x06_P2.54mm_Vertical
Changed lines of the file:
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@@
 			)
 		)
-		(property "Footprint" "Connector_PinHeader_2.54mm:PinHeader_1x06_P2.54mm_Vertical"
+		(property "Footprint" "Connector_PinSocket_2.54mm:PinSocket_1x06_P2.54mm_Vertical"
 			(at 63.5 81.28 0)
 			(effects
@@
 			)
 		)
-		(property "Footprint" "Connector_PinHeader_2.54mm:PinHeader_1x06_P2.54mm_Vertical"
+		(property "Footprint" "Connector_PinSocket_2.54mm:PinSocket_1x06_P2.54mm_Vertical"
 			(at 63.5 127 0)
 			(effects
@@
 		(exclude_from_sim no)
 		(in_bom yes)
-		(on_board yes)
+		(on_board no)
 		(dnp no)
 		(fields_autoplaced yes)
@@
 			)
 		)
-		(property "Footprint" "Connector_PinHeader_2.54mm:PinHeader_1x06_P2.54mm_Vertical"
+		(property "Footprint" "Connector_PinSocket_2.54mm:PinSocket_1x06_P2.54mm_Vertical"
 			(at 76.2 100.33 0)
 			(effects
@@
 			)
 		)
-		(property "Footprint" "Connector_PinHeader_2.54mm:PinHeader_1x06_P2.54mm_Vertical"
+		(property "Footprint" "Connector_PinSocket_2.54mm:PinSocket_1x06_P2.54mm_Vertical"
 			(at 110.49 129.54 0)
 			(effects
@@
 			)
 		)
-		(property "Footprint" "Connector_PinHeader_2.54mm:PinHeader_1x06_P2.54mm_Vertical"
+		(property "Footprint" "Connector_PinSocket_2.54mm:PinSocket_1x06_P2.54mm_Vertical"
 			(at 63.5 120.65 0)
 			(effects
@@
 			)
 		)
-		(property "Footprint" "Connector_PinHeader_2.54mm:PinHeader_1x06_P2.54mm_Vertical"
+		(property "Footprint" "Connector_PinSocket_2.54mm:PinSocket_1x06_P2.54mm_Vertical"
 			(at 63.5 114.3 0)
 			(effects

Commit message: pcb 2 routing in progress
Connections:
- net Drive CV Input: now also J17.2 (Pin_2); no longer J17.1 (Pin_1)
- net at R113.1, RV27.2: now also J17.1 (Pin_1); no longer J17.3 (Pin_3)
- net at RV25.2, U9.12 (+): now also J17.3 (Pin_3); no longer J17.2 (Pin_2)
Changed lines of the file:
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@@
 		(lib_id "SynthStuff:Conn_01x06_PinHeader")
 		(at 63.5 81.28 270)
-		(unit 1)
+		(unit 2)
 		(exclude_from_sim no)
 		(in_bom yes)
@@
 				(path "/58f4306d-5387-4983-bb08-41a2313fd315/76f3ab41-888d-43b6-843a-2a995f9c890b"
 					(reference "J17")
-					(unit 1)
+					(unit 2)
 				)
 			)
@@
 		(lib_id "SynthStuff:Conn_01x06_PinHeader")
 		(at 76.2 100.33 90)
-		(unit 2)
+		(unit 3)
 		(exclude_from_sim no)
 		(in_bom yes)
@@
 				(path "/58f4306d-5387-4983-bb08-41a2313fd315/76f3ab41-888d-43b6-843a-2a995f9c890b"
 					(reference "J17")
-					(unit 2)
+					(unit 3)
 				)
 			)
@@
 		(lib_id "SynthStuff:Conn_01x06_PinHeader")
 		(at 110.49 129.54 90)
-		(unit 3)
+		(unit 1)
 		(exclude_from_sim no)
 		(in_bom yes)
@@
 				(path "/58f4306d-5387-4983-bb08-41a2313fd315/76f3ab41-888d-43b6-843a-2a995f9c890b"
 					(reference "J17")
-					(unit 3)
-				)
-			)
+					(unit 1)
+				)
+			)

Commit message: Adjusted pin header connections
Parts:
- RV26: Function (none) -> Drive A VCA Center
Changed lines of the file:
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@@
 		(on_board no)
 		(dnp no)
-		(fields_autoplaced yes)
 		(property "Reference" "RV26"
 			(at 224.79 100.3299 0)
@@
 			)
 		)
+		(property "Function" "Drive A VCA Center"
+			(at 239.522 101.6 0)
+			(effects
+				(font
+					(size 1.27 1.27)
+					(thickness 0.254)
+					(bold yes)
+					(italic yes)
+				)
+			)
+		)

Commit message: Changed VCA CV summing stage feedback to 100k
Parts:
- R112: value 82k -> 100k
Changed lines of the file:
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@@
 			)
 		)
-		(property "Value" "82k"
+		(property "Value" "100k"
 			(at 138.43 110.49 90)
 			(effects

Commit message: Synchronized changes from PCB 1 to PCB 2 schematic
Parts:
- removed R101: 1k, Resistor_THT:R_Axial_DIN0207_L6.3mm_D2.5mm_P7.62mm_Horizontal, symbol Device:R_US
Connections:
- net Output: now also R99.1, U9.8
Changed lines of the file:
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@@
-	(wire
-		(pts
-			(xy 257.81 50.8) (xy 266.7 50.8)
-		)
-		(stroke
-			(width 0)
-			(type default)
-		)
-	)
 	(wire
 		(pts
@@
 	(wire
 		(pts
-			(xy 246.38 50.8) (xy 250.19 50.8)
+			(xy 246.38 50.8) (xy 266.7 50.8)
 		)
 		(stroke
@@
 					(unit 1)
 				)
-			)
-		)
-	)
-	(symbol
-		(lib_id "Device:R_US")
-		(at 254 50.8 270)
-		(unit 1)
-		(exclude_from_sim no)
-		(in_bom yes)
-		(on_board no)
-		(dnp no)
-		(fields_autoplaced yes)
-		(property "Reference" "R101"
-			(at 254 44.45 90)
-			(effects
-				(font
-					(size 1.27 1.27)
-				)
-			)
-		)
-		(property "Value" "1k"
-			(at 254 46.99 90)
-			(effects
-				(font
-					(size 1.27 1.27)
-				)
-			)
-		)
-		(property "Footprint" "Resistor_THT:R_Axial_DIN0207_L6.3mm_D2.5mm_P7.62mm_Horizontal"
-			(at 253.746 51.816 90)
-			(effects
-				(font
-					(size 1.27 1.27)
-				)
-				(hide yes)
-			)
-		)
-		(property "Datasheet" "~"
-			(at 254 50.8 0)
-			(effects
-				(font
-					(size 1.27 1.27)
-				)
-				(hide yes)
-			)
-		)
-		(property "Description" "Resistor, US symbol"
-			(at 254 50.8 0)
-			(effects
-				(font
-					(size 1.27 1.27)
-				)
-				(hide yes)
-			)
-		)
-		(property "Function" ""
-			(at 254 50.8 0)
-			(effects
-				(font
-					(size 1.27 1.27)
-				)
-			)
-		)
-		(pin "1"
-		)
-		(pin "2"
-		)
-		(instances
-			(project "DMH_Dual_VCF_Diode_Ladder_Mk2_PCB_1"
-				(path "/58f4306d-5387-4983-bb08-41a2313fd315/76f3ab41-888d-43b6-843a-2a995f9c890b"
-					(reference "R101")
-					(unit 1)
-				)

Commit message: Mistakes found during assembly
Parts:
- R111: value 20k -> 10k
Changed lines of the file:
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@@
 			)
 		)
-		(property "Value" "20k"
+		(property "Value" "10k"
 			(at 104.14 115.5699 0)
 			(effects
