File: DMH_Dual_VCF_Diode_Ladder_Mk2_PCB_2/CV_Processing.kicad_sch (KiCad schematic)
At the start: 58 parts, among them J15 Conn_01x08_PinHeader, J16 Conn_01x08_PinHeader, SW10 SW_DPDT_OnOn, SW7 SW_SPDT_OnOffOn, SW9 SW_SPDT_OnOffOn, U7 TL074, U8 TL074

Commit message: Finished Mk2.0
Connections:
- net at R24.2, RV31.2: now also SW9.1 (A); no longer SW9.3 (C)
- net at SW7.1 (A): now also R10.2, RV19.2; no longer R10.1
- net at R24.1: now also SW9.3 (C); no longer SW9.1 (A)
- new net: R10.1, SW7.3 (C)
Other:
- moved on the sheet: SW7, SW9
Changed lines of the file:
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@@
 	(symbol
 		(lib_id "Switch:SW_SPDT")
-		(at 90.17 114.3 180)
+		(at 90.17 114.3 0)
+		(mirror y)
 		(unit 1)
 		(exclude_from_sim no)
@@
 		(dnp no)
 		(property "Reference" "SW7"
+			(at 90.17 109.22 0)
+			(effects
+				(font
+					(size 1.27 1.27)
+				)
+			)
+		)
+		(property "Value" "SW_SPDT_OnOffOn"
 			(at 90.17 119.38 0)
-			(effects
-				(font
-					(size 1.27 1.27)
-				)
-			)
-		)
-		(property "Value" "SW_SPDT_OnOffOn"
-			(at 90.17 109.22 0)
 			(effects
 				(font
@@
 		)
 		(property "Datasheet" "~"
-			(at 90.17 106.68 0)
+			(at 90.17 121.92 0)
 			(effects
 				(font
@@
 		)
 		(property "Function" "CV 3 Amt"
-			(at 90.424 121.666 0)
+			(at 90.424 106.934 0)
 			(effects
 				(font
@@
 	(symbol
 		(lib_id "Switch:SW_SPDT")
-		(at 90.17 241.3 180)
+		(at 90.17 241.3 0)
+		(mirror y)
 		(unit 1)
 		(exclude_from_sim no)
@@
 		(dnp no)
 		(property "Reference" "SW9"
+			(at 90.17 236.22 0)
+			(effects
+				(font
+					(size 1.27 1.27)
+				)
+			)
+		)
+		(property "Value" "SW_SPDT_OnOffOn"
 			(at 90.17 246.38 0)
-			(effects
-				(font
-					(size 1.27 1.27)
-				)
-			)
-		)
-		(property "Value" "SW_SPDT_OnOffOn"
-			(at 90.17 236.22 0)
 			(effects
 				(font
@@
 		)
 		(property "Datasheet" "~"
-			(at 90.17 233.68 0)
+			(at 90.17 248.92 0)
 			(effects
 				(font
@@
 		)
 		(property "Function" "CV 3 Amt"
-			(at 90.424 248.666 0)
-			(effects
-				(font
+			(at 90.424 233.934 0)
+			(effects
+				(font

Commit message: Re-exported Gerbers
Parts:
- SW10: Function Link -> Link CV
Changed lines of the file:
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@@
 			)
 		)
-		(property "Function" "Link"
+		(property "Function" "Link CV"
 			(at 158.75 155.448 0)
 			(effects
