File: DMH_Dual_VCF_Diode_Ladder_Mk2_PCB_2/Core_Circuit_A.kicad_sch (KiCad schematic)
At the start: 41 parts, among them J19 Conn_01x04_PinHeader, SW1 SW_SPDT, SW2 SW_SPDT, SW3 SW_SPDT, U3 TL074, U5 TL074

Commit message: Adjusted pin header connections
Parts:
- RV13: Function Resonance Intensity -> Res A Intensity
Changed lines of the file:
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@@
 			)
 		)
-		(property "Function" "Resonance Intensity"
+		(property "Function" "Res A Intensity"
 			(at 209.55 23.876 90)
 			(effects

Commit message: Synchronized changes from PCB 1 to PCB 2 schematic
Parts:
- added unit 5 of J19
- added unit 6 of J19
- added R142: 51k, Resistor_THT:R_Axial_DIN0207_L6.3mm_D2.5mm_P7.62mm_Horizontal, symbol Device:R_US
- added R143: 1k, Resistor_THT:R_Axial_DIN0207_L6.3mm_D2.5mm_P7.62mm_Horizontal, symbol Device:R_US
- J19: value Conn_01x04_PinHeader -> Conn_01x06_PinHeader; footprint Connector_PinSocket_2.54mm:PinSocket_1x04_P2.54mm_Vertical -> (none); symbol SynthStuff:Conn_01x04_PinHeader -> SynthStuff:Conn_01x06_PinHeader
- R39: value 1k -> 100k
- R41: value 47K -> 100k
Connections:
- net GND: now also J19.6 (Pin_6), R143.1
- net Raw Output: now also R142.2; no longer U3.6 (-)
- net at D13.1 (K), D14.2 (A), R38.2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: now also J19.5 (Pin_5)
- new net: R142.1, R143.2, U3.6 (-)

Commit message: Updated PCB 2 with validated features
Parts:
- J19: footprint (none) -> Connector_PinSocket_2.54mm:PinSocket_1x06_P2.54mm_Vertical
Changed lines of the file:
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@@
 			)
 		)
-		(property "Footprint" ""
+		(property "Footprint" "Connector_PinSocket_2.54mm:PinSocket_1x06_P2.54mm_Vertical"
 			(at 146.05 81.28 0)
 			(effects
@@
 			)
 		)
-		(property "Footprint" ""
+		(property "Footprint" "Connector_PinSocket_2.54mm:PinSocket_1x06_P2.54mm_Vertical"
 			(at 74.93 41.91 0)
 			(effects
@@
 			)
 		)
-		(property "Footprint" ""
+		(property "Footprint" "Connector_PinSocket_2.54mm:PinSocket_1x06_P2.54mm_Vertical"
 			(at 203.2 25.4 0)
 			(effects
@@
 			)
 		)
-		(property "Footprint" ""
+		(property "Footprint" "Connector_PinSocket_2.54mm:PinSocket_1x06_P2.54mm_Vertical"
 			(at 228.6 50.8 0)
 			(effects
@@
 			)
 		)
-		(property "Footprint" ""
+		(property "Footprint" "Connector_PinSocket_2.54mm:PinSocket_1x06_P2.54mm_Vertical"
 			(at 134.62 114.3 0)
 			(effects
@@
 			)
 		)
-		(property "Footprint" ""
+		(property "Footprint" "Connector_PinSocket_2.54mm:PinSocket_1x06_P2.54mm_Vertical"
 			(at 88.9 69.85 0)
 			(effects
